File: powerboard-hw/powerboard-v1/powerboard-v1.kicad_pcb (KiCad board)
At the start: 2 copper layers, 16 x 45.7 mm, 25 parts, among them J1 Conn_01x02, J2 PWR, J3 SIG, Q1 AO3401A, Q2 AO3400A, SW1 OS102011MA1Q, U1 TPS62842DGRR

Commit message: fix: JLCPCB-ready silkscreen and ordering notes
- Silkscreen text stroke 0.12 -> 0.15 mm (JLCPCB minimum line width).
- JLCJLCJLCJLC placeholder on the bottom for the order number.
- JP1 labels BUCK / 3V3 on the top only (bottom copy ran into J3's label).
- README: JLCPCB order settings, assembly and first power-up checklist,
  output capacitance limit (3 ... 40 uF effective) for the load.
- Regenerated Gerbers, drill, position file and images.

ERC: 0. DRC: 0 violations, 0 unconnected, schematic parity OK.

Co-Authored-By: Claude Opus 5.5 <noreply@anthropic.com>
Other:
- board text added: "JLCJLCJLCJLC"

Commit message: fix: SW1 switches the converter enable instead of the battery line
SW1 (C&K OS102011MA1Q) is rated 100 mA and sat in series with the
battery, which limited the module to about 120 mA. It now drives the
TPS62842 EN pin (net BUCK_EN): middle pin to EN, left pin to +BATT,
right pin to GND. Only the EN input current flows through it; the load
current goes J1 -> F1 -> D1 -> converter. F1 (500 mA hold) is now the
lowest limit, about 600 mA at 3.3 V.

ON/OFF direction from the C&K OS series datasheet (position 1 = 1-2,
position 2 = 2-3: the slider connects the middle pin to the outer pin
on its side): slider left = 2-3 = ON, slider right = 1-2 = OFF, printed
as ON / OFF at the two ends of the switch. OFF shuts the converter down
(25 nA typ.) and discharges +3V3; +BATT stays connected.

PCB: F1 connects straight to D1; BUCK_EN runs along the right edge with
one short B.Cu hop under the +BATT feed to J2. Schematic notes and
README (switch table, current limits, power-up steps) updated.

ERC: 0. DRC: 0 violations, 0 unconnected, schematic parity OK.

Co-Authored-By: Claude Opus 5.5 <noreply@anthropic.com>
Connections:
- F1 pad 2: Net-(F1-Pad2) -> Net-(D1-A)
- SW1 pad 1: Net-(F1-Pad2) -> GND
- SW1 pad 2: Net-(D1-A) -> /BUCK_EN
- SW1 pad 3: (no net) -> +BATT
- U1 pad 5: +BATT -> /BUCK_EN
Routing:
- net /BUCK_EN: track 0.00 -> 35.3 mm, vias 0 -> 2
- net Net-(F1-Pad2): track 4.92 -> 0.00 mm
- net +BATT: track 42.6 -> 44.4 mm
- net Net-(D1-A): track 4.35 -> 2.92 mm
- net GND: vias 15 -> 14
Other:
- board text added: "OFF"
- board text added: "ON"

Commit message: fix: battery divider R1/R2 100k instead of 1M
The divider is switched off by Q1 between measurements, so it no longer
needs megaohm values. With 100k/100k the settling of C17 (150 nF)
drops from tau = 75 ms to 7.5 ms: about 65 ms before the ADC reading
instead of 0.6 s. Current while measuring is about 37 uA, the charge
per measurement is lower than before (about 4 uC vs 7 uC).

R3/R4 stay 1M. Board geometry unchanged (tracks, vias, pads, silk,
fills identical); only the values in schematic, BOM, position file and
Gerber attributes change. Schematic notes and README timing updated.

ERC: 0. DRC: 0 violations, 0 unconnected, schematic parity OK.

Co-Authored-By: Claude Opus 5.5 <noreply@anthropic.com>
Parts:
- R1, R2: value 1M -> 100k
